Commit message: 1

File: robot_specific_config/abb_irb14000_moveit_config/config/abb_irb14000_macro.srdf.xacro (robot description, xacro)
@@ -7,4 +7,10 @@
     <group name="left_arm">
       <chain base_link="robl_base_link" tip_link="robl_tool0" />
+    </group>
+    <group name="right_gripper">
+      <joint name="grpr_half_aperture_joint" />
+    </group>
+    <group name="left_gripper">
+      <joint name="grpl_half_aperture_joint" />
     </group>
     <group_state name="all_zero" group="right_arm">
@@ -26,5 +32,7 @@
       <joint name="robl_joint_7" value="0" />
     </group_state>
-    <virtual_joint type="floating" parent_frame="world" child_link="base_link" />
+    <virtual_joint name="world_joint" type="floating" parent_frame="world" child_link="base_link" />
+    <end_effector name="right_gripper_eef" parent_link="robr_tool0" group="right_gripper" parent_group="right_arm" />
+    <end_effector name="left_gripper_eef" parent_link="robl_tool0" group="left_gripper" parent_group="left_arm" />
     <disable_collisions link1="robr_base_link" link2="robr_link_1" reason="Adjacent" />
     <disable_collisions link1="robr_link_1" link2="robr_link_2" reason="Adjacent" />
@@ -41,4 +49,10 @@
     <disable_collisions link1="robl_link_5" link2="robl_link_6" reason="Adjacent" />
     <disable_collisions link1="robl_link_6" link2="robl_link_7" reason="Adjacent" />
+    <disable_collisions link1="robr_tool0" link2="grpr_base" reason="Adjacent" />
+    <disable_collisions link1="grpr_base" link2="grpr_finger_r" reason="Adjacent" />
+    <disable_collisions link1="grpr_base" link2="grpr_finger_l" reason="Adjacent" />
+    <disable_collisions link1="robl_tool0" link2="grpl_base" reason="Adjacent" />
+    <disable_collisions link1="grpl_base" link2="grpl_finger_r" reason="Adjacent" />
+    <disable_collisions link1="grpl_base" link2="grpl_finger_l" reason="Adjacent" />
   </xacro:macro>
 </robot>
